Commit message: chore: modified quadrotor mass, arm length, and motor positions

File: resources/robots/quad/quad.urdf (robot description, URDF)
Before this commit: robot quadrotor, 9 links, 8 joints
Links:
- link arm_motor_0: geometry visual cylinder length=0.466 radius=0.01
- link arm_motor_1: geometry visual cylinder length=0.466 radius=0.01
- link arm_motor_2: geometry visual cylinder length=0.466 radius=0.01
- link arm_motor_3: geometry visual cylinder length=0.466 radius=0.01
- link base_link: mass 0.225 -> 2.36
Joints:
- joint base_link_to_motor_0: origin xyz=0.13 -0.13 0.0 rpy=0.0 0.0 0.0 -> xyz=0.23 -0.23 0.0 rpy=0.0 0.0 0.0
- joint base_link_to_motor_1: origin xyz=-0.13 -0.13 0.0 rpy=0.0 0.0 0.0 -> xyz=-0.23 -0.23 0.0 rpy=0.0 0.0 0.0
- joint base_link_to_motor_2: origin xyz=-0.13 0.13 0.0 rpy=0.0 0.0 0.0 -> xyz=-0.23 0.23 0.0 rpy=0.0 0.0 0.0
- joint base_link_to_motor_3: origin xyz=0.13 0.13 0.0 rpy=0.0 0.0 0.0 -> xyz=0.23 0.23 0.0 rpy=0.0 0.0 0.0
